Commit message: Mecanum drive support and IMU fix (#2)
* Feat: Diff drive setup working with odom and joy_node

* Feat: Added mecanum drive support with arguments to select between diffdrive and mecanum

* Seperated Teleop and controls into different launch files

* Added FeedForward argument for robots without feedback

* feat: Update int_brain_description and int_brain_system packages

- Added dependency on int_brain_hardware in package.xml of int_brain_description.
- Introduced a new link (pcb_link) and joint (pcb_joint) in the URDF file for the PCB component.
- Replaced the imu_calibrate executable with imu_feedback_node in CMakeLists.txt and updated installation targets.
- Increased the update rate for the controller manager in controllers.yaml.
- Added a new EKF configuration file (ekf.yaml) for robot localization.
- Updated pltjg_ctrl_dbg.xml for improved UI layout and plot configurations.
- Enhanced teleop_joy_params.yaml to include parameters for the new imu_feedback_node.
- Modified view.rviz to include visualization settings for the new pcb_link.
- Updated system.launch.py to include EKF node and remap topics for odometry.
- Added imu_feedback_node to teleop_joy.launch.py for feedback based on IMU data.
- Updated package.xml of int_brain_system to include additional dependencies for robot localization and control.
- Removed obsolete IMU calibration and covariance nodes from src directory.
- Implemented imu_feedback.cpp to provide haptic feedback based on IMU linear acceleration.

* Fix order in which data comes from pcb

* Update: Better response. removed gravity effect

* fix: adjust update rate and enhance teleop launch with RViz integration

* - Removed Buad rate configuration.
-  Fix encoder calculation api
- Update teleop params

* fix: clarify rpm_desired_ variable comment to specify units in rad/s

* Feat: Smoother and Responsive teleop

* Fix Wheel order

* Added .gitignore

* feat: add custom effort controllers and system identifier node

- Implemented custom effort controllers with a new SystemIdentifier class.
- Added necessary CMake and package configuration files.
- Created XML and YAML configurations for the controller.
- Developed a system identifier node for publishing commands and handling responses.

* WIP: send config Frames during on_configure phase and params parsing from urdf.
____
BUG: FF1 is not being updated in STM correctly.

* feat: send config

* xacro param name fix

* hardware port possible fix

* fix: invert connection check for comms in on_configure

* attempt to migrate to `LibSerial::SerialStream`

* Fix pcb orientation and imu frame

* Fix axis +ve dir

* Improved cmd_vel visualization

* add keyboard teleop launch file

---------

Co-authored-by: Eccentric Orange <eccentric.orange2@gmail.com>

File: int_brain_description/urdf/int_brain.xacro (robot description, xacro)
@@ -3,4 +3,5 @@
   <xacro:arg name="controllers_yaml" default="" />
   <xacro:arg name="sim" default="true" />
+  <xacro:arg name="is_feedforward" default="false" />
   <xacro:include filename="$(find int_brain_description)/urdf/macros.xacro" />
   <xacro:include filename="$(find int_brain_description)/urdf/materials.xacro" />
@@ -35,9 +36,35 @@
     </collision>
   </link>
+  <link name="pcb_link">
+    <inertial>
+      <origin xyz="0 0 -0.001" rpy="0 0 0" />
+      <mass value="0.02" />
+      <inertia ixx="1e-05" iyy="1e-05" izz="1e-05" ixy="0.0" iyz="0.0" ixz="0.0" />
+    </inertial>
+    <visual>
+      <origin xyz="-0.1 0.06 -0.001" rpy="0 0 0" />
+      <geometry>
+        <mesh filename="file://$(find int_brain_description)/meshes/int-brain-pcb.dae"
+          scale="0.001 0.001 0.001" />
+      </geometry>
+    </visual>
+    <collision>
+      <origin xyz="-0.1 0.06 -0.001" rpy="0 0 0" />
+      <geometry>
+        <mesh filename="file://$(find int_brain_description)/meshes/int-brain-pcb.dae"
+          scale="0.001 0.001 0.001" />
+      </geometry>
+    </collision>
+  </link>
+  <joint name="pcb_joint" type="fixed">
+    <parent link="base_link" />
+    <child link="pcb_link" />
+    <origin xyz="0 0 0.01" rpy="0 0 3.1414" />
+  </joint>
   <link name="imu_link" />
   <joint name="imu_joint" type="fixed">
-    <parent link="base_link" />
+    <parent link="pcb_link" />
     <child link="imu_link" />
-    <origin xyz="0 0 0.061" rpy="3.1414 0 1.5707" />
+    <origin xyz="-0.0072 -0.0123 0" rpy="0 3.1414 -1.5707" />
   </joint>
   <joint name="base_footprint_to_base_link" type="fixed">

File: int_brain_description/urdf/ros2_control_hardware.xacro (robot description, xacro)
@@ -4,12 +4,58 @@
         <hardware>
             <plugin>int_brain_hardware/IntBrainHardware</plugin>
-            <param name="device_addr">/dev/int-brain-315936583034</param>
-            <param name="baud_rate">230400</param>
-            <param name="timeout_ms">500</param>
+            <param name="device_addr">/dev/int-brain-316436653034</param>
+            <param name="timeout_ms">100</param>
+            <param name="is_feedforward">$(arg is_feedforward)</param>
+            <!-- IMU settings -->
+            <param name="imu_usage">true</param>
+            <param name="imu_sensor_fusion">true</param>
+            <param name="imu_sensor_fusion_frequency">100</param>
+            <!-- Encoder settings -->
+            <param name="encoder_usage">true</param>
+            <param name="encoder_velocity_calculation">true</param>
+            <param name="encoder_velocity_calculation_frequency">100</param>
+            <param name="encoder_cpr">1320</param>
+            <!-- Motor current measurement settings -->
+            <param name="motor_current_meas_on_off">true</param>
+            <param name="motor_current_meas_frequency">100</param>
+            <!-- Battery voltage measurement settings -->
+            <param name="battery_voltage_meas_on_off">true</param>
+            <param name="battery_voltage_meas_rate">10</param>
+            <!-- Motor closed loop control settings -->
+            <param name="motor_control_mode">pid_feed_forward</param>
+            <param name="motor_controller_frequency">200</param>
         </hardware>
+        <joint name="front_right_shaft_joint">
+            <command_interface name="velocity" />
+            <state_interface name="position" />
+            <state_interface name="velocity" />
+            <param name="kp">6.0</param>
+            <param name="ki">3.5</param>
+            <param name="kd">-0.005</param>
+            <param name="kd_filter_coeff">10.0</param>
+            <param name="ff0">1.004187035789131</param>
+            <param name="ff1">0.12866352232164302</param>
+        </joint>
+        <joint name="rear_right_shaft_joint">
+            <command_interface name="velocity" />
+            <state_interface name="position" />
+            <state_interface name="velocity" />
+            <param name="kp">6.0</param>
+            <param name="ki">3.5</param>
+            <param name="kd">-0.005</param>
+            <param name="kd_filter_coeff">10.0</param>
+            <param name="ff0">0.966311070657699</param>
+            <param name="ff1">0.15775862872871882</param>
+        </joint>
         <joint name="front_left_shaft_joint">
             <command_interface name="velocity" />
             <state_interface name="position" />
             <state_interface name="velocity" />
+            <param name="kp">6.0</param>
+            <param name="ki">3.5</param>
+            <param name="kd">-0.005</param>
+            <param name="kd_filter_coeff">10.0</param>
+            <param name="ff0">1.0200673342777509</param>
+            <param name="ff1">-0.3682036005229734</param>
         </joint>
         <joint name="rear_left_shaft_joint">
@@ -17,14 +63,10 @@
             <state_interface name="position" />
             <state_interface name="velocity" />
-        </joint>
-        <joint name="front_right_shaft_joint">
-            <command_interface name="velocity" />
-            <state_interface name="position" />
-            <state_interface name="velocity" />
-        </joint>
-        <joint name="rear_right_shaft_joint">
-            <command_interface name="velocity" />
-            <state_interface name="position" />
-            <state_interface name="velocity" />
+            <param name="kp">5.0</param>
+            <param name="ki">3.5</param>
+            <param name="kd">-0.005</param>
+            <param name="kd_filter_coeff">10.0</param>
+            <param name="ff0">1.008908105064786</param>
+            <param name="ff1">-0.2470694664139883</param>
         </joint>
         <sensor name="imu_sensor">

Commit message: Imu data reception (#6)
* Refactor IMU data requests to seperate acceleration and gyro data handling
* Bump botspeak version
* Conform with ICM 20948 IC frame convention
* FIX: Bug in data acquisition
* Improve IMU data error logging by specifying data type in error messages

File: int_brain_description/urdf/int_brain.xacro (robot description, xacro)
@@ -66,5 +66,5 @@
     <parent link="pcb_link" />
     <child link="imu_link" />
-    <origin xyz="-0.0072 -0.0123 0" rpy="0 3.1414 -1.5707" />
+    <origin xyz="-0.0072 -0.0123 0" rpy="0 0 1.5707" />
   </joint>
   <joint name="base_footprint_to_base_link" type="fixed">
