Commit message: it works

File: jr_bot_description/urdf/jr_bot.ros2_control.xacro (robot description, xacro)
@@ -1,5 +1,5 @@
 <?xml version="1.0"?>
 <robot xmlns:xacro="http://www.ros.org/wiki/xacro">
-    <xacro:macro name="jr_bot_ros2_control" params="device_addr:='/dev/ttyUSB0'">
+    <xacro:macro name="jr_bot_ros2_control" params="device_addr:='/dev/ttyACM0'">
         <ros2_control name="JrBotSystem" type="system">
             <hardware>

File: jr_bot_description/urdf/jr_bot.xacro (robot description, xacro)
@@ -2,5 +2,5 @@
 <robot name="jr_bot" xmlns:xacro="http://www.ros.org/wiki/xacro">
     <xacro:include filename="$(find jr_bot_description)/urdf/jr_bot.ros2_control.xacro" />
-    <xacro:jr_bot_ros2_control device_addr="/dev/ttyUSB0" />
+    <xacro:jr_bot_ros2_control device_addr="/dev/ttyACM0" />
     <material name="black">
         <color rgba="0.1 0.1 0.1 1.0"/>

Commit message: kinda works

File: jr_bot_description/urdf/jr_bot.ros2_control.xacro (robot description, xacro)
@@ -31,8 +31,4 @@
                 <command_interface name="state"/>
             </gpio>
-            <gpio name="tof_sweep">
-                <state_interface name="distance"/>
-                <state_interface name="angle"/>
-            </gpio>
             <gpio name="ir_sensor_left">
                 <state_interface name="state"/>
@@ -41,4 +37,10 @@
                 <state_interface name="state"/>
             </gpio>
+            <joint name="tof_sweep_distance">
+                <state_interface name="position"/>
+            </joint>
+            <joint name="tof_sweep_angle">
+                <state_interface name="position"/>
+            </joint>
         </ros2_control>
     </xacro:macro>

File: jr_bot_description/urdf/jr_bot.xacro (robot description, xacro)
@@ -114,4 +114,17 @@
         <origin xyz="0.10 0 0.035" rpy="0 0 0"/>
     </joint>
+    <link name="tof_distance_link" />
+    <joint name="tof_sweep_distance" type="prismatic">
+        <parent link="tof_link"/>
+        <child link="tof_distance_link"/>
+        <axis xyz="1 0 0"/>
+        <limit lower="0.0" upper="10.0" effort="0" velocity="0"/>
+    </joint>
+    <link name="tof_angle_link" />
+    <joint name="tof_sweep_angle" type="continuous">
+        <parent link="tof_link"/>
+        <child link="tof_angle_link"/>
+        <axis xyz="0 0 1"/>
+    </joint>
     <link name="imu_link">
         <visual>

Commit message: TOF works

File: jr_bot_description/urdf/jr_bot.ros2_control.xacro (robot description, xacro)
@@ -37,10 +37,8 @@
                 <state_interface name="state"/>
             </gpio>
-            <joint name="tof_sweep_distance">
-                <state_interface name="position"/>
-            </joint>
-            <joint name="tof_sweep_angle">
-                <state_interface name="position"/>
-            </joint>
+            <sensor name="tof_sweep">
+                <state_interface name="distance"/>
+                <state_interface name="angle"/>
+            </sensor>
         </ros2_control>
     </xacro:macro>
